Commit message: urdf

File: arm.urdf (robot description, URDF)
Before this commit: robot my_arm, 1 links, 0 joints
Links:
- added link link_servo_holder_0; visual box size=0.02 0.057 0.05
- added link link_servo_holder_1; visual box size=0.04 0.057 0.025
Joints:
- added joint joint_base_2_servo_0: type fixed, parent base_link, child link_servo_holder_0
- added joint servo0: type continuous, parent link_servo_holder_0, child link_servo_holder_1, origin xyz=0.0 -0.01 0.0645 rpy=0.0 0.0 0.0, axis 0.0 0.0 1.0
